Commit message: gazebo controller

File: rx90_description/urdf/rx90.urdf (robot description, URDF)
Before this commit: robot RX90, 5 links, 4 joints
Links:
- added link RX90_ELBOW, mass 1; collision mesh filename=package://rx90_description/meshes/stl/RX-90_ELBOW.stl scale=0.001 0.001 0.001; visual mesh filename=package://rx90_description/meshes/stl/RX-90_ELBOW.stl scale=0.001 0.001 0.001
- added link RX90_FLANGE, mass 1; collision mesh filename=package://rx90_description/meshes/stl/RX-90_FLANGE.stl scale=0.001 0.001 0.001; visual mesh filename=package://rx90_description/meshes/stl/RX-90_FLANGE.stl scale=0.001 0.001 0.001
- added link RX90_FOREARM, mass 1; collision mesh filename=package://rx90_description/meshes/stl/RX-90_FOREARM.stl scale=0.001 0.001 0.001; visual mesh filename=package://rx90_description/meshes/stl/RX-90_FOREARM.stl scale=0.001 0.001 0.001
- added link RX90_WRIST, mass 1; collision mesh filename=package://rx90_description/meshes/stl/RX-90_WRIST.stl scale=0.001 0.001 0.001; visual mesh filename=package://rx90_description/meshes/stl/RX-90_WRIST.stl scale=0.001 0.001 0.001
- link RX90_ARM: mass None -> 1
- link RX90_BARREL: mass None -> 1
- link RX90_BASE: mass None -> 1
- link RX90_SHOULDER: mass None -> 1
Joints:
- added joint RX90_ELBOW_JOINT: type continuous, parent RX90_ARM, child RX90_ELBOW, origin xyz=-0.255 0 -0.46 rpy=0 0 0
- added joint RX90_FLANGE_JOINT: type continuous, parent RX90_WRIST, child RX90_FLANGE, origin xyz=-0.006 -0.1015 -0.009 rpy=0 0 ${-pi/2}
- added joint RX90_FOREARM_JOINT: type continuous, parent RX90_ELBOW, child RX90_FOREARM, origin xyz=0 0 0 rpy=0 0 ${-pi/2}
- added joint RX90_WRIST_JOINT: type continuous, parent RX90_FOREARM, child RX90_WRIST, origin xyz=0.52 0 0 rpy=0 0 ${pi/2}
- joint RX90_ARM_JOINT: origin xyz=0 0 -1 rpy=0 ${pi/2} ${pi/2} -> xyz=0 0 -0.301 rpy=0 ${pi/2} ${pi/2}
- joint RX90_BASE_JOINT: origin xyz=0 0 5.3 rpy=0 0 0 -> xyz=0 0 1.005 rpy=0 0 0
- joint RX90_SHOULDER_JOINT: origin xyz=0 0 3 rpy=0 ${pi/2} 0 -> xyz=0 0 0.41 rpy=0 ${pi/2} 0

File: rx90_description/urdf/rx90.xacro (robot description, xacro)
@@ -11,5 +11,5 @@
 <!--BRAZOOOOOOOOOOOOOOOOOOOO-->
 <!-- Joint 0 -->
-     <link name="RX90_BARREL">
+   <link name="RX90_BARREL">
       <visual>
          <geometry>
@@ -65,9 +65,9 @@
        <parent link="RX90_BARREL" />
        <child link="RX90_BASE" />
-       <origin rpy="0 0 0" xyz="0 0 5.3" />
+       <origin rpy="0 0 0" xyz="0 0 1.005" />
     </joint>
     <link name="RX90_SHOULDER">
        <visual>
-	<origin rpy="${pi/2} 0 ${pi}" xyz="0 0 0" />
+	<origin rpy="0 ${-pi/2} ${pi/2}" xyz="0.122 0 0" />
           <geometry>
              <mesh filename="package://rx90_description/meshes/stl/RX-90_SHOULDER.stl" scale="0.001 0.001 0.001" />
@@ -75,5 +75,5 @@
        </visual>
 	<collision>
-        <origin rpy="${pi/2} 0 ${pi}" xyz="0 0 0" />
+        <origin rpy="0 ${-pi/2} ${pi/2}" xyz="0.122 0 0" />
             <geometry>
               <mesh filename="package://rx90_description/meshes/stl/RX-90_SHOULDER.stl" scale="0.001 0.001 0.001" />
@@ -93,5 +93,5 @@
        <parent link="RX90_BASE" />
        <child link="RX90_SHOULDER" />
-       <origin rpy="0 ${pi/2} 0" xyz="0 0 3" />
+       <origin rpy="0 ${pi/2} 0" xyz="0 0 0.41" />
     </joint>
 <link name="RX90_ARM">
@@ -121,5 +121,117 @@
        <parent link="RX90_SHOULDER" />
        <child link="RX90_ARM" />
-       <origin rpy="0 ${pi/2} ${pi/2}" xyz="0 0 -1" />
+       <origin rpy="0 ${pi/2} ${pi/2}" xyz="0 0 -0.301" />
+    </joint>
+    <link name="RX90_ELBOW">
+       <visual>
+	<origin rpy="${-pi/2} ${-pi/2} ${-pi/2}" xyz="-0.021 0.14 0" />
+          <geometry>
+             <mesh filename="package://rx90_description/meshes/stl/RX-90_ELBOW.stl" scale="0.001 0.001 0.001" />
+          </geometry>
+       </visual>
+	<collision>
+        <origin rpy="${-pi/2} ${-pi/2} ${-pi/2}" xyz="-0.021 0.14 0" />
+            <geometry>
+              <mesh filename="package://rx90_description/meshes/stl/RX-90_ELBOW.stl" scale="0.001 0.001 0.001" />
+            </geometry>
+       </collision>
+       <selfCollide>true</selfCollide>
+	<inertial>
+        <origin xyz="0 0 0" rpy="0 0 0" />
+        <mass value="1" />
+        <inertia
+          ixx="1.0" ixy="0.0" ixz="0.0"
+          iyy="1.0" iyz="0.0"
+          izz="1.0" />
+    </inertial>
+    </link>
+    <joint name="RX90_ELBOW_JOINT" type="continuous">
+       <parent link="RX90_ARM" />
+       <child link="RX90_ELBOW" />
+       <origin rpy="0 0 0" xyz="-0.255 0 -0.46" />
+    </joint>
+  <link name="RX90_FOREARM">
+       <visual>
+	<origin rpy="${pi} ${-pi/2} 0" xyz="0.355 0.1 -0.05" />
+          <geometry>
+             <mesh filename="package://rx90_description/meshes/stl/RX-90_FOREARM.stl" scale="0.001 0.001 0.001" />
+          </geometry>
+       </visual>
+	<collision>
+        <origin rpy="${pi} ${-pi/2} 0" xyz="0.355 0.1 -0.05" />
+            <geometry>
+              <mesh filename="package://rx90_description/meshes/stl/RX-90_FOREARM.stl" scale="0.001 0.001 0.001" />
+            </geometry>
+       </collision>
+       <selfCollide>true</selfCollide>
+	<inertial>
+        <origin xyz="0 0 0" rpy="0 0 0" />
+        <mass value="1" />
+        <inertia
+          ixx="1.0" ixy="0.0" ixz="0.0"
+          iyy="1.0" iyz="0.0"
+          izz="1.0" />
+    </inertial>
+    </link>
+    <joint name="RX90_FOREARM_JOINT" type="continuous">
+       <parent link="RX90_ELBOW" />
+       <child link="RX90_FOREARM" />
+       <origin rpy="0 0 ${-pi/2}" xyz="0 0 0" />
+    </joint>
+      <link name="RX90_WRIST">
+       <visual>
+	<origin rpy="${pi/2} 0 ${-pi/2}" xyz="-0.007 0 -0.01" />
+          <geometry>
+             <mesh filename="package://rx90_description/meshes/stl/RX-90_WRIST.stl" scale="0.001 0.001 0.001" />
+          </geometry>
+       </visual>
+	<collision>
+        <origin rpy="${pi/2} 0 ${-pi/2}" xyz="-0.007 0 -0.01" />
+            <geometry>
+              <mesh filename="package://rx90_description/meshes/stl/RX-90_WRIST.stl" scale="0.001 0.001 0.001" />
+            </geometry>
+       </collision>
+       <selfCollide>true</selfCollide>
+	<inertial>
+        <origin xyz="0 0 0" rpy="0 0 0" />
+        <mass value="1" />
+        <inertia
+          ixx="1.0" ixy="0.0" ixz="0.0"
+          iyy="1.0" iyz="0.0"
+          izz="1.0" />
+    </inertial>
+    </link>
+    <joint name="RX90_WRIST_JOINT" type="continuous">
+       <parent link="RX90_FOREARM" />
+       <child link="RX90_WRIST" />
+       <origin rpy="0 0 ${pi/2}" xyz="0.52 0 0" />
+    </joint>
+          <link name="RX90_FLANGE">
+       <visual>
+	<origin rpy="0 ${pi/2} 0" xyz="0 0 0" />
+          <geometry>
+             <mesh filename="package://rx90_description/meshes/stl/RX-90_FLANGE.stl" scale="0.001 0.001 0.001" />
+          </geometry>
+       </visual>
+	<collision>
+        <origin rpy="0 ${pi/2} 0" xyz="0 0 -0.009" />
+            <geometry>
+              <mesh filename="package://rx90_description/meshes/stl/RX-90_FLANGE.stl" scale="0.001 0.001 0.001" />
+            </geometry>
+       </collision>
+       <selfCollide>true</selfCollide>
+	<inertial>
+        <origin xyz="0 0 0" rpy="0 0 0" />
+        <mass value="1" />
+        <inertia
+          ixx="1.0" ixy="0.0" ixz="0.0"
+          iyy="1.0" iyz="0.0"
+          izz="1.0" />
+    </inertial>
+    </link>
+    <joint name="RX90_FLANGE_JOINT" type="continuous">
+       <parent link="RX90_WRIST" />
+       <child link="RX90_FLANGE" />
+       <origin rpy="0 0 ${-pi/2}" xyz="-0.006 -0.1015 -0.009" />
     </joint>
 <selfCollide>true</selfCollide>
@@ -147,3 +259,43 @@
     </actuator>
   </transmission>
+  <transmission name="tran_RX90_ELBOW_JOINT">
+    <type>transmission_interface/SimpleTransmission</type>
+    <joint name="RX90_ELBOW_JOINT">
+      <hardwareInterface>hardware_interface/EffortJointInterface</hardwareInterface>
+    </joint>
+    <actuator name="motor_RX90_ELBOW_JOINT">
+      <hardwareInterface>hardware_interface/EffortJointInterface</hardwareInterface>
+      <mechanicalReduction>1</mechanicalReduction>
+    </actuator>
+  </transmission>
+  <transmission name="tran_RX90_FOREARM_JOINT">
+    <type>transmission_interface/SimpleTransmission</type>
+    <joint name="RX90_FOREARM_JOINT">
+      <hardwareInterface>hardware_interface/EffortJointInterface</hardwareInterface>
+    </joint>
+    <actuator name="motor_RX90_FOREARM_JOINT">
+      <hardwareInterface>hardware_interface/EffortJointInterface</hardwareInterface>
+      <mechanicalReduction>1</mechanicalReduction>
+    </actuator>
+  </transmission>
+  <transmission name="tran_RX90_WRIST_JOINT">
+    <type>transmission_interface/SimpleTransmission</type>
+    <joint name="RX90_WRIST_JOINT">
+      <hardwareInterface>hardware_interface/EffortJointInterface</hardwareInterface>
+    </joint>
+    <actuator name="motor_RX90_WRIST_JOINT">
+      <hardwareInterface>hardware_interface/EffortJointInterface</hardwareInterface>
+      <mechanicalReduction>1</mechanicalReduction>
+    </actuator>
+  </transmission>
+  <transmission name="tran_RX90_FLANGE_JOINT">
+    <type>transmission_interface/SimpleTransmission</type>
+    <joint name="RX90_FLANGE_JOINT">
+      <hardwareInterface>hardware_interface/EffortJointInterface</hardwareInterface>
+    </joint>
+    <actuator name="motor_RX90_FLANGE_JOINT">
+      <hardwareInterface>hardware_interface/EffortJointInterface</hardwareInterface>
+      <mechanicalReduction>1</mechanicalReduction>
+    </actuator>
+  </transmission>
 </robot>

Commit message: world and controllers updated

File: rx90_description/urdf/rx90.urdf (robot description, URDF)
Before this commit: robot RX90, 9 links, 8 joints
Links:
- added link RX90_LGRIPPER, mass 1; collision box size=0.02 0.045 0.01; visual box size=0.02 0.045 0.01
- added link RX90_RGRIPPER, mass 1; collision box size=0.02 0.045 0.01; visual box size=0.02 0.045 0.01
Joints:
- added joint RX90_LGRIPPER_JOINT: type prismatic, parent RX90_FLANGE, child RX90_LGRIPPER, origin xyz=0.025 0.03 0 rpy=0 0 ${-pi/2}, limit lower=0 upper=0.1 effort=1000.0 velocity=0.5
- added joint RX90_RGRIPPER_JOINT: type prismatic, parent RX90_FLANGE, child RX90_RGRIPPER, origin xyz=0.025 -0.03 0 rpy=0 0 ${-pi/2}, limit lower=-0.1 upper=0 effort=1000.0 velocity=0.5

File: rx90_description/urdf/rx90.xacro (robot description, xacro)
@@ -235,4 +235,62 @@
        <origin rpy="0 0 ${-pi/2}" xyz="-0.006 -0.1015 -0.009" />
     </joint>
+              <link name="RX90_LGRIPPER">
+       <visual>
+	<origin rpy="0 0 0" xyz="0 0 0" />
+          <geometry>
+            <box size="0.02 0.045 0.01"/>
+          </geometry>
+       </visual>
+	<collision>
+        <origin rpy="0 0 0" xyz="0 0 0" />
+            <geometry>
+              <box size="0.02 0.045 0.01"/>
+            </geometry>
+       </collision>
+       <selfCollide>true</selfCollide>
+	<inertial>
+        <origin xyz="0 0 0" rpy="0 0 0" />
+        <mass value="1" />
+        <inertia
+          ixx="1.0" ixy="0.0" ixz="0.0"
+          iyy="1.0" iyz="0.0"
+          izz="1.0" />
+    </inertial>
+    </link>
+    <joint name="RX90_LGRIPPER_JOINT" type="prismatic">
+    <limit effort="1000.0" lower="0" upper="0.1" velocity="0.5"/>
+       <parent link="RX90_FLANGE" />
+       <child link="RX90_LGRIPPER" />
+       <origin rpy="0 0 ${-pi/2}" xyz="0.025 0.03 0" />
+    </joint>
+ <link name="RX90_RGRIPPER">
+       <visual>
+	<origin rpy="0 0 0" xyz="0 0 0" />
+          <geometry>
+            <box size="0.02 0.045 0.01"/>
+          </geometry>
+       </visual>
+	<collision>
+        <origin rpy="0 0 0" xyz="0 0 0" />
+            <geometry>
+              <box size="0.02 0.045 0.01"/>
+            </geometry>
+       </collision>
+       <selfCollide>true</selfCollide>
+	<inertial>
+        <origin xyz="0 0 0" rpy="0 0 0" />
+        <mass value="1" />
+        <inertia
+          ixx="1.0" ixy="0.0" ixz="0.0"
+          iyy="1.0" iyz="0.0"
+          izz="1.0" />
+    </inertial>
+    </link>
+    <joint name="RX90_RGRIPPER_JOINT" type="prismatic">
+    <limit effort="1000.0" lower="-0.1" upper="0" velocity="0.5"/>
+       <parent link="RX90_FLANGE" />
+       <child link="RX90_RGRIPPER" />
+       <origin rpy="0 0 ${-pi/2}" xyz="0.025 -0.03 0" />
+    </joint>
 <selfCollide>true</selfCollide>
 <!--BRAZOOOOOOOOOOOOOOOOOOOOooooooooooooooooooooooooooooooooooooooo-->
@@ -299,3 +357,23 @@
     </actuator>
   </transmission>
+    <transmission name="tran_RX90_LGRIPPER_JOINT">
+    <type>transmission_interface/SimpleTransmission</type>
+    <joint name="RX90_LGRIPPER_JOINT">
+      <hardwareInterface>hardware_interface/EffortJointInterface</hardwareInterface>
+    </joint>
+    <actuator name="motor_RX90_LGRIPPER_JOINT">
+      <hardwareInterface>hardware_interface/EffortJointInterface</hardwareInterface>
+      <mechanicalReduction>1</mechanicalReduction>
+    </actuator>
+  </transmission>
+    <transmission name="tran_RX90_RGRIPPER_JOINT">
+    <type>transmission_interface/SimpleTransmission</type>
+    <joint name="RX90_RGRIPPER_JOINT">
+      <hardwareInterface>hardware_interface/EffortJointInterface</hardwareInterface>
+    </joint>
+    <actuator name="motor_RX90_RGRIPPER_JOINT">
+      <hardwareInterface>hardware_interface/EffortJointInterface</hardwareInterface>
+      <mechanicalReduction>1</mechanicalReduction>
+    </actuator>
+  </transmission>
 </robot>

Commit message: publisher and client

File: rx90_description/urdf/rx90.urdf (robot description, URDF)
Before this commit: robot RX90, 11 links, 10 joints
Links:
- added link RX90_MGRIPPER, mass 1; collision box size=0.02 0.045 0.01; visual box size=0.02 0.045 0.01
Joints:
- added joint RX90_MGRIPPER_JOINT: type prismatic, parent RX90_FLANGE, child RX90_MGRIPPER, origin xyz=0.025 0 -0.035 rpy=0 ${pi/2} ${-pi/2}, limit lower=-0.05 upper=0 effort=1000.0 velocity=0.5
- joint RX90_LGRIPPER_JOINT: origin xyz=0.025 0.03 0 rpy=0 0 ${-pi/2} -> xyz=0.025 0.03 0.015 rpy=0 0 ${-pi/2}
- joint RX90_RGRIPPER_JOINT: origin xyz=0.025 -0.03 0 rpy=0 0 ${-pi/2} -> xyz=0.025 -0.03 0.015 rpy=0 0 ${-pi/2}

File: rx90_description/urdf/rx90.xacro (robot description, xacro)
@@ -238,5 +238,5 @@
        <origin rpy="0 0 ${-pi/2}" xyz="-0.006 -0.1015 -0.009" />
     </joint>
-              <link name="RX90_LGRIPPER">
+          <link name="RX90_LGRIPPER">
        <visual>
 	<origin rpy="0 0 0" xyz="0 0 0" />
@@ -265,5 +265,5 @@
        <parent link="RX90_FLANGE" />
        <child link="RX90_LGRIPPER" />
-       <origin rpy="0 0 ${-pi/2}" xyz="0.025 0.03 0" />
+       <origin rpy="0 0 ${-pi/2}" xyz="0.025 0.03 0.015" />
     </joint>
  <link name="RX90_RGRIPPER">
@@ -294,7 +294,35 @@
        <parent link="RX90_FLANGE" />
        <child link="RX90_RGRIPPER" />
-       <origin rpy="0 0 ${-pi/2}" xyz="0.025 -0.03 0" />
-    </joint>
-<selfCollide>true</selfCollide>
+       <origin rpy="0 0 ${-pi/2}" xyz="0.025 -0.03 0.015" />
+    </joint>
+     <link name="RX90_MGRIPPER">
+       <visual>
+	<origin rpy="0 0 0" xyz="0 0 0" />
+          <geometry>
+            <box size="0.02 0.045 0.01"/>
+          </geometry>
+       </visual>
+	<collision>
+        <origin rpy="0 0 0" xyz="0 0 0" />
+            <geometry>
+              <box size="0.02 0.045 0.01"/>
+            </geometry>
+       </collision>
+       <selfCollide>true</selfCollide>
+	<inertial>
+        <origin xyz="0 0 0" rpy="0 0 0" />
+        <mass value="1" />
+        <inertia
+          ixx="1.0" ixy="0.0" ixz="0.0"
+          iyy="1.0" iyz="0.0"
+          izz="1.0" />
+    </inertial>
+    </link>
+    <joint name="RX90_MGRIPPER_JOINT" type="prismatic">
+    <limit effort="1000.0" lower="-0.05" upper="0" velocity="0.5"/>
+       <parent link="RX90_FLANGE" />
+       <child link="RX90_MGRIPPER" />
+       <origin rpy="0 ${pi/2} ${-pi/2}" xyz="0.025 0 -0.035" />
+    </joint>
 <!--BRAZOOOOOOOOOOOOOOOOOOOOooooooooooooooooooooooooooooooooooooooo-->
   <!-- Base Link -->
@@ -380,3 +408,13 @@
     </actuator>
   </transmission>
+      <transmission name="tran_RX90_MGRIPPER_JOINT">
+    <type>transmission_interface/SimpleTransmission</type>
+    <joint name="RX90_MGRIPPER_JOINT">
+      <hardwareInterface>hardware_interface/EffortJointInterface</hardwareInterface>
+    </joint>
+    <actuator name="motor_RX90_MGRIPPER_JOINT">
+      <hardwareInterface>hardware_interface/EffortJointInterface</hardwareInterface>
+      <mechanicalReduction>1</mechanicalReduction>
+    </actuator>
+  </transmission>
 </robot>

Commit message: joint limits

File: rx90_description/urdf/rx90.urdf (robot description, URDF)
Before this commit: robot RX90, 12 links, 11 joints
Joints:
- joint RX90_ARM_JOINT: limit (none) -> lower=-0.82 upper=3.96 effort=10000 velocity=3.4906; type continuous -> revolute
- joint RX90_ELBOW_JOINT: limit (none) -> lower=-0.917 upper=4.057 effort=10000 velocity=4.9916; type continuous -> revolute
- joint RX90_FLANGE_JOINT: limit (none) -> lower=-4.712 upper=4.712 effort=10000 velocity=10.122; type continuous -> revolute
- joint RX90_FOREARM_JOINT: limit (none) -> lower=-4.712 upper=4.712 effort=10000 velocity=6.9987; type continuous -> revolute
- joint RX90_SHOULDER_JOINT: limit (none) -> lower=-2.7925 upper=2.7925 effort=10000 velocity=4.1189; type continuous -> revolute
- joint RX90_WRIST_JOINT: limit (none) -> lower=-2 upper=1.8325 effort=10000 velocity=5.585; type continuous -> revolute

File: rx90_description/urdf/rx90.xacro (robot description, xacro)
@@ -93,5 +93,6 @@
     </inertial>
     </link>
-    <joint name="RX90_SHOULDER_JOINT" type="continuous">
+    <joint name="RX90_SHOULDER_JOINT" type="revolute">
+    <limit effort="10000" lower="-2.7925" upper="2.7925" velocity="4.1189"/>
        <parent link="RX90_BASE" />
        <child link="RX90_SHOULDER" />
@@ -121,5 +122,6 @@
     </inertial>
     </link>
-    <joint name="RX90_ARM_JOINT" type="continuous">
+    <joint name="RX90_ARM_JOINT" type="revolute">
+    <limit effort="10000" lower="-0.82" upper="3.96" velocity="3.4906"/>
        <parent link="RX90_SHOULDER" />
        <child link="RX90_ARM" />
@@ -149,5 +151,6 @@
     </inertial>
     </link>
-    <joint name="RX90_ELBOW_JOINT" type="continuous">
+    <joint name="RX90_ELBOW_JOINT" type="revolute">
+    <limit effort="10000" lower="-0.917" upper="4.057" velocity="4.9916"/>
        <parent link="RX90_ARM" />
        <child link="RX90_ELBOW" />
@@ -177,5 +180,6 @@
     </inertial>
     </link>
-    <joint name="RX90_FOREARM_JOINT" type="continuous">
+    <joint name="RX90_FOREARM_JOINT" type="revolute">
+    <limit effort="10000" lower="-4.712" upper="4.712" velocity="6.9987"/>
        <parent link="RX90_ELBOW" />
        <child link="RX90_FOREARM" />
@@ -205,5 +209,6 @@
     </inertial>
     </link>
-    <joint name="RX90_WRIST_JOINT" type="continuous">
+    <joint name="RX90_WRIST_JOINT" type="revolute">
+    <limit effort="10000" lower="-2" upper="1.8325" velocity="5.585"/>
        <parent link="RX90_FOREARM" />
        <child link="RX90_WRIST" />
@@ -233,5 +238,6 @@
     </inertial>
     </link>
-    <joint name="RX90_FLANGE_JOINT" type="continuous">
+    <joint name="RX90_FLANGE_JOINT" type="revolute">
+    <limit effort="10000" lower="-4.712" upper="4.712" velocity="10.122"/>
        <parent link="RX90_WRIST" />
        <child link="RX90_FLANGE" />

Commit message: Moveit config package

File: rx90_description/urdf/rx90.urdf (robot description, URDF)
Before this commit: robot RX90, 12 links, 11 joints
Links:
- link RX90_ARM: mass 1 -> 51.266495
- link RX90_BASE: mass 1 -> 23.085357
- link RX90_ELBOW: mass 1 -> 19.754401
- link RX90_FLANGE: mass 1 -> 0.038484
- link RX90_FOREARM: mass 1 -> 15.287896
- link RX90_LGRIPPER: mass 1 -> 0.038484
- link RX90_MGRIPPER: mass 1 -> 0.038484
- link RX90_RGRIPPER: mass 1 -> 0.038484
- link RX90_SHOULDER: mass 1 -> 45.357763
- link RX90_WRIST: mass 1 -> 0.548088
Joints:
- joint RX90_LGRIPPER_JOINT: limit lower=0 upper=0.1 effort=1000.0 velocity=0.5 -> lower=-100000 upper=1 effort=100000.0 velocity=20
- joint RX90_MGRIPPER_JOINT: limit lower=-0.05 upper=0 effort=1000.0 velocity=0.5 -> lower=-100000 upper=1 effort=100000.0 velocity=20
- joint RX90_RGRIPPER_JOINT: limit lower=-0.1 upper=0 effort=1000.0 velocity=0.5 -> lower=-100000 upper=1 effort=100000.0 velocity=20
