Commit message: DOUBLE ARMS YEAHHHHHHHHH

File: rx90_description/urdf/rx90.xacro (robot description, xacro)
@@ -19,5 +19,5 @@
             <mesh filename="package://rx90_description/meshes/stl/RX-90_BARREL.stl" scale="0.001 0.001 0.001" />
          </geometry>
-          <origin rpy="${pi/2} 0 0" xyz="0 0 0" />
+          <origin rpy="${pi/2} 0 0" xyz= "0 0 0"/>
       </visual>
       <collision>

Commit message: .

File: rx90_description/urdf/rx90.xacro (robot description, xacro)
@@ -19,5 +19,5 @@
             <mesh filename="package://rx90_description/meshes/stl/RX-90_BARREL.stl" scale="0.001 0.001 0.001" />
          </geometry>
-          <origin rpy="${pi/2} 0 0" xyz= "0 0 0"/>
+          <origin rpy="${pi/2} ${pi/2} ${pi/2}" xyz= "0 0 0"/>
       </visual>
       <collision>

File: rx90_description/urdf/rx90_floor.xacro (robot description, xacro)
@@ -13,5 +13,5 @@
     <link name="RX90_BASE">
        <visual>
-	<origin rpy="${pi/2} 0 0" xyz="0 0 0" />
+	<origin rpy="${pi/2} 0 ${pi/2}" xyz="0 0 0" />
           <geometry>
              <mesh filename="package://rx90_description/meshes/stl/RX-90_BASE.stl" scale="0.001 0.001 0.001" />
