Commit message: Gazebo simulation working

File: rx90_description/urdf/rx90_floor.xacro (robot description, xacro)
@@ -7,6 +7,5 @@
   <!-- Import Rviz colors -->
   <xacro:include filename="$(find rx90_description)/urdf/materials.xacro" />
-  <link name="world"/>
-<!--link name="base_link"/-->
+<link name="base_link"/>
 <!--BRAZOOOOOOOOOOOOOOOOOOOO-->
 <!-- Joint 0 -->
@@ -34,5 +33,5 @@
     </link>
     <joint name="RX90_BASE_JOINT" type="fixed">
-       <parent link="world" />
+       <parent link="base_link" />
        <child link="RX90_BASE" />
        <origin rpy="0 0 0" xyz="0 0 0.083" />

File: rx90_description/urdf/rx90_floor_noinertia.xacro (robot description, xacro)
@@ -13,5 +13,5 @@
     <link name="RX90_BASE">
        <visual>
-	<origin rpy="${pi/2} 0 0" xyz="0 0 0" />
+	<origin rpy="${pi/2} 0 ${pi/2}" xyz="0 0 0" />
           <geometry>
              <mesh filename="package://rx90_description/meshes/stl/RX-90_BASE.stl" scale="0.001 0.001 0.001" />
@@ -26,9 +26,9 @@
        <selfCollide>true</selfCollide>
 	<inertial>
-       <mass value="1"/>
+       <mass value="0.1"/>
           <origin xyz="0.0 0.00 0.0" rpy="0.0 0.0 0.0"/>
-          <inertia ixx="1"  ixy="1"  ixz="1"
-                   iyx="1"  iyy="1"  iyz="1"
-                   izx="1"  izy="1"  izz="1"/>
+          <inertia ixx="0.1"  ixy="0.1"  ixz="0.1"
+                   iyx="0.1"  iyy="0.1"  iyz="0.1"
+                   izx="0.1"  izy="0.1"  izz="0.1"/>
     </inertial>
     </link>
@@ -53,9 +53,9 @@
        <selfCollide>true</selfCollide>
 	<inertial>
-      <mass value="1"/>
+      <mass value="0.1"/>
       <origin xyz="0.0 0.00 0.0" rpy="0.0 0.0 0.0"/>
-          <inertia ixx="1"  ixy="1"  ixz="1"
-                   iyx="1"  iyy="1"  iyz="1"
-                   izx="1"  izy="1"  izz="1"/>
+          <inertia ixx="0.1"  ixy="0.1"  ixz="0.1"
+                   iyx="0.1"  iyy="0.1"  iyz="0.1"
+                   izx="0.1"  izy="0.1"  izz="0.1"/>
     </inertial>
     </link>
@@ -81,9 +81,9 @@
        <selfCollide>true</selfCollide>
 	<inertial>
-        <mass value="1"/>
+        <mass value="0.1"/>
   <origin xyz="0.0 0.00 0.0" rpy="0.0 0.0 0.0"/>
-          <inertia ixx="1"  ixy="1"  ixz="1"
-                   iyx="1"  iyy="1"  iyz="1"
-                   izx="1"  izy="1"  izz="1"/>
+          <inertia ixx="0.1"  ixy="0.1"  ixz="0.1"
+                   iyx="0.1"  iyy="0.1"  iyz="0.1"
+                   izx="0.1"  izy="0.1"  izz="0.1"/>
     </inertial>
     </link>
@@ -109,9 +109,9 @@
        <selfCollide>true</selfCollide>
 	<inertial>
-  <mass value="1"/>
+  <mass value="0.1"/>
         <origin xyz="0.0 0.00 0.0" rpy="0.0 0.0 0.0"/>
-          <inertia ixx="1"  ixy="1"  ixz="1"
-                   iyx="1"  iyy="1"  iyz="1"
-                   izx="1"  izy="1"  izz="1"/>
+          <inertia ixx="0.1"  ixy="0.1"  ixz="0.1"
+                   iyx="0.1"  iyy="0.1"  iyz="0.1"
+                   izx="0.1"  izy="0.1"  izz="0.1"/>
     </inertial>
     </link>
@@ -137,13 +137,13 @@
        <selfCollide>true</selfCollide>
 	<inertial>
-        <mass value="1"/>
+        <mass value="0.1"/>
           <origin xyz="0.0 0.00 0.0" rpy="0.0 0.0 0.0"/>
-          <inertia ixx="1"  ixy="1"  ixz="1"
-                   iyx="1"  iyy="1"  iyz="1"
-                   izx="1"  izy="1"  izz="1"/>
+          <inertia ixx="0.1"  ixy="0.1"  ixz="0.1"
+                   iyx="0.1"  iyy="0.1"  iyz="0.1"
+                   izx="0.1"  izy="0.1"  izz="0.1"/>
     </inertial>
     </link>
     <joint name="RX90_FOREARM_JOINT" type="revolute">
-    <limit effort="10000" lower="-4.712" upper="4.712" velocity="6.9987"/>
+    <limit effort="10000" lower="-3.14" upper="3.14" velocity="6.9987"/>
        <parent link="RX90_ELBOW" />
        <child link="RX90_FOREARM" />
@@ -165,9 +165,9 @@
        <selfCollide>true</selfCollide>
 	<inertial>
-       <mass value="1"/>
+       <mass value="0.1"/>
          <origin xyz="0.0 0.00 0.0" rpy="0.0 0.0 0.0"/>
-          <inertia ixx="1"  ixy="1"  ixz="1"
-                   iyx="1"  iyy="1"  iyz="1"
-                   izx="1"  izy="1"  izz="1"/>
+          <inertia ixx="0.1"  ixy="0.1"  ixz="0.1"
+                   iyx="0.1"  iyy="0.1"  iyz="0.1"
+                   izx="0.1"  izy="0.1"  izz="0.1"/>
     </inertial>
     </link>
@@ -194,9 +194,9 @@
 	<inertial>
          <origin xyz="0 0 0" rpy="0 0 0" />
-         <mass value="1"/>
+         <mass value="0.1"/>
         <origin xyz="0.0 0.00 0.0" rpy="0.0 0.0 0.0"/>
-          <inertia ixx="1"  ixy="1"  ixz="1"
-                   iyx="1"  iyy="1"  iyz="1"
-                   izx="1"  izy="1"  izz="1"/>
+          <inertia ixx="0.1"  ixy="0.1"  ixz="0.1"
+                   iyx="0.1"  iyy="0.1"  iyz="0.1"
+                   izx="0.1"  izy="0.1"  izz="0.1"/>
     </inertial>
     </link>
@@ -222,9 +222,9 @@
        <selfCollide>true</selfCollide>
 	<inertial>
-        <mass value="1" />
+        <mass value="0.1" />
   <origin xyz="0.0 0.00 0.0" rpy="0.0 0.0 0.0"/>
-          <inertia ixx="1"  ixy="1"  ixz="1"
-                   iyx="1"  iyy="1"  iyz="1"
-                   izx="1"  izy="1"  izz="1"/>
+          <inertia ixx="0.1"  ixy="0.1"  ixz="0.1"
+                   iyx="0.1"  iyy="0.1"  iyz="0.1"
+                   izx="0.1"  izy="0.1"  izz="0.1"/>
     </inertial>
     </link>
@@ -251,8 +251,8 @@
 	<inertial>
        <origin xyz="0 0 0" rpy="0 0 0" />
-        <mass value="1" />
-          <inertia ixx="1"  ixy="1"  ixz="1"
-                   iyx="1"  iyy="1"  iyz="1"
-                   izx="1"  izy="1"  izz="1"/>
+        <mass value="0.1" />
+          <inertia ixx="0.1"  ixy="0.1"  ixz="0.1"
+                   iyx="0.1"  iyy="0.1"  iyz="0.1"
+                   izx="0.1"  izy="0.1"  izz="0.1"/>
     </inertial>
     </link>
@@ -279,8 +279,8 @@
 	<inertial>
        <origin xyz="0 0 0" rpy="0 0 0" />
-        <mass value="1" />
-          <inertia ixx="1"  ixy="1"  ixz="1"
-                   iyx="1"  iyy="1"  iyz="1"
-                   izx="1"  izy="1"  izz="1"/>
+        <mass value="0.1" />
+          <inertia ixx="0.1"  ixy="0.1"  ixz="0.1"
+                   iyx="0.1"  iyy="0.1"  iyz="0.1"
+                   izx="0.1"  izy="0.1"  izz="0.1"/>
     </inertial>
     </link>

Commit message: gazebo sim

File: rx90_description/urdf/rx90_floor.xacro (robot description, xacro)
@@ -7,5 +7,5 @@
   <!-- Import Rviz colors -->
   <xacro:include filename="$(find rx90_description)/urdf/materials.xacro" />
-<link name="base_link"/>
+<link name="world"/>
 <!--BRAZOOOOOOOOOOOOOOOOOOOO-->
 <!-- Joint 0 -->
@@ -33,5 +33,5 @@
     </link>
     <joint name="RX90_BASE_JOINT" type="fixed">
-       <parent link="base_link" />
+       <parent link="world" />
        <child link="RX90_BASE" />
        <origin rpy="0 0 0" xyz="0 0 0.083" />
