Commit message: base_link

File: rx90_description/urdf/rx90_floor_baselink.xacro (robot description, xacro)
@@ -7,49 +7,23 @@
   <!-- Import Rviz colors -->
   <xacro:include filename="$(find rx90_description)/urdf/materials.xacro" />
+    <!--NO SE USA EL PLUGIN DESDE QUE PODEMOS SUBSCRIBRNOS A LOS TOPICOS DE GAZEBO-->
 <!--gazebo>
-  <plugin name="rx90_publisher" filename="librx90_publisher.so"/>
-  </gazebo-->
-  <!-- Used for fixing robot to Gazebo 'base_link' -->
-  <link name="world"/>
+<plugin name="contact_plugin" filename="libcontact_plugin.so">
+</plugin>
+</gazebo-->
+  <link name="base_link"/>
+<!--link name="base_link"/-->
 <!--BRAZOOOOOOOOOOOOOOOOOOOO-->
 <!-- Joint 0 -->
-   <link name="RX90_BARREL">
-      <visual>
-         <geometry>
-            <mesh filename="package://rx90_description/meshes/stl/RX-90_BARREL.stl" scale="0.001 0.001 0.001" />
-         </geometry>
-          <origin rpy="${pi/2} 0 0" xyz= "0 0 0"/>
-      </visual>
-      <collision>
+    <link name="RX90_BASE">
+       <visual>
+	<origin rpy="${pi/2} 0 ${pi/2}" xyz="0 0 0" />
+          <geometry>
+             <mesh filename="package://rx90_description/meshes/stl/RX-90_BASE.stl" scale="0.001 0.001 0.001" />
+          </geometry>
+       </visual>
+	<collision>
         <origin rpy="${pi/2} 0 0" xyz="0 0 0" />
             <geometry>
-              <mesh filename="package://rx90_description/meshes/stl/RX-90_BARREL.stl" scale="0.001 0.001 0.001" />
-            </geometry>
-       </collision>
-       <selfCollide>true</selfCollide>
-	<inertial>
-        <origin xyz="0 0 0" rpy="0 0 0" />
-        <mass value="1" />
-        <inertia
-          ixx="1.0" ixy="0.0" ixz="0.0"
-          iyy="1.0" iyz="0.0"
-          izz="1.0" />
-    </inertial>
-   </link>
-   <joint name="RX90_BARREL_JOINT" type="fixed">
-      <parent link="world" />
-      <child link="RX90_BARREL" />
-      <origin rpy="0 0 0" xyz="0 0 0" />
-   </joint>
-    <link name="RX90_BASE">
-       <visual>
-	<origin rpy="${pi/2} 0 0" xyz="0 0 0" />
-          <geometry>
-             <mesh filename="package://rx90_description/meshes/stl/RX-90_BASE.stl" scale="0.001 0.001 0.001" />
-          </geometry>
-       </visual>
-	<collision>
-        <origin rpy="${pi/2} 0 0" xyz="0 0 0" />
-            <geometry>
               <mesh filename="package://rx90_description/meshes/stl/RX-90_BASE.stl" scale="0.001 0.001 0.001" />
             </geometry>
@@ -57,15 +31,15 @@
        <selfCollide>true</selfCollide>
 	<inertial>
-        <mass value="23.085357"/>
-          <origin xyz="0.007579 0.000017 0.180670" rpy="0.0 0.0 0.0"/>
-          <inertia ixx="0.343576" ixy="-0.000062" ixz="-0.002079"
-                                  iyy="0.336217"  iyz="-0.000014"
-                                                  izz="0.334050"/>
+       <mass value="0.1"/>
+          <origin xyz="0.0 0.00 0.0" rpy="0.0 0.0 0.0"/>
+          <inertia ixx="0.1"  ixy="0.1"  ixz="0.1"
+                   iyx="0.1"  iyy="0.1"  iyz="0.1"
+                   izx="0.1"  izy="0.1"  izz="0.1"/>
     </inertial>
     </link>
     <joint name="RX90_BASE_JOINT" type="fixed">
-       <parent link="RX90_BARREL" />
+       <parent link="base_link" />
        <child link="RX90_BASE" />
-       <origin rpy="0 0 0" xyz="0 0 1.005" />
+       <origin rpy="0 0 0" xyz="0 0 0.083" />
     </joint>
     <link name="RX90_SHOULDER">
@@ -84,9 +58,9 @@
        <selfCollide>true</selfCollide>
 	<inertial>
-        <mass value="45.357763"/>
-          <origin xyz="0.085479 -0.002547 -0.040488" rpy="0.0 0.0 0.0"/>
-          <inertia ixx="0.839141" ixy="0.022637" ixz="0.162457"
-                                  iyy="1.030146" iyz="0.027416"
-                                                  izz="1.064698"/>
+      <mass value="0.1"/>
+      <origin xyz="0.0 0.00 0.0" rpy="0.0 0.0 0.0"/>
+          <inertia ixx="0.1"  ixy="0.1"  ixz="0.1"
+                   iyx="0.1"  iyy="0.1"  iyz="0.1"
+                   izx="0.1"  izy="0.1"  izz="0.1"/>
     </inertial>
     </link>
@@ -112,16 +86,16 @@
        <selfCollide>true</selfCollide>
 	<inertial>
-        <mass value="51.266495"/>
-          <origin xyz="-0.000002 0.264164 0.347704" rpy="0.0 0.0 0.0"/>
-          <inertia ixx="5.272800" ixy="0.000010" ixz="0.000017"
-                                  iyy="5.536809" iyz="-0.008261"
-                                                  izz="0.486191"/>
+        <mass value="0.1"/>
+  <origin xyz="0.0 0.00 0.0" rpy="0.0 0.0 0.0"/>
+          <inertia ixx="0.1"  ixy="0.1"  ixz="0.1"
+                   iyx="0.1"  iyy="0.1"  iyz="0.1"
+                   izx="0.1"  izy="0.1"  izz="0.1"/>
     </inertial>
     </link>
     <joint name="RX90_ARM_JOINT" type="revolute">
-    <limit effort="10000" lower="-0.82" upper="3.96" velocity="3.4906"/>
+    <limit effort="10000" lower="-2.39" upper="2.39" velocity="3.4906"/>
        <parent link="RX90_SHOULDER" />
        <child link="RX90_ARM" />
-       <origin rpy="0 ${pi/2} ${pi/2}" xyz="0 0 -0.301" />
+       <origin rpy="0 ${pi/2} 0" xyz="0 0 -0.301" />
     </joint>
     <link name="RX90_ELBOW">
@@ -140,16 +114,16 @@
        <selfCollide>true</selfCollide>
 	<inertial>
-        <mass value="19.754401"/>
-          <origin xyz="-0.000255 0.016478 -0.003819" rpy="0.0 0.0 0.0"/>
-          <inertia ixx="0.249388" ixy="-0.004901" ixz="0.004825"
-                                  iyy="0.211780"  iyz="0.000574"
-                                                  izz="0.238488"/>
+  <mass value="0.1"/>
+        <origin xyz="0.0 0.00 0.0" rpy="0.0 0.0 0.0"/>
+          <inertia ixx="0.1"  ixy="0.1"  ixz="0.1"
+                   iyx="0.1"  iyy="0.1"  iyz="0.1"
+                   izx="0.1"  izy="0.1"  izz="0.1"/>
     </inertial>
     </link>
     <joint name="RX90_ELBOW_JOINT" type="revolute">
-    <limit effort="10000" lower="-0.917" upper="4.057" velocity="4.9916"/>
+    <limit effort="10000" lower="-2.487" upper="2.487" velocity="4.9916"/>
        <parent link="RX90_ARM" />
        <child link="RX90_ELBOW" />
-       <origin rpy="0 0 0" xyz="-0.255 0 -0.46" />
+       <origin rpy="${pi/2} 0 0" xyz="-0.255 0 -0.46" />
     </joint>
   <link name="RX90_FOREARM">
@@ -168,13 +142,13 @@
        <selfCollide>true</selfCollide>
 	<inertial>
-       <mass value="15.287896"/>
-          <origin xyz="-0.015515 0.000164 0.340348" rpy="0.0 0.0 0.0"/>
-          <inertia ixx="0.331593" ixy="0.000055" ixz="-0.010688"
-                                  iyy="0.320895" iyz="0.000058"
-                                                  izz="0.086557"/>
+        <mass value="0.1"/>
+          <origin xyz="0.0 0.00 0.0" rpy="0.0 0.0 0.0"/>
+          <inertia ixx="0.1"  ixy="0.1"  ixz="0.1"
+                   iyx="0.1"  iyy="0.1"  iyz="0.1"
+                   izx="0.1"  izy="0.1"  izz="0.1"/>
     </inertial>
     </link>
     <joint name="RX90_FOREARM_JOINT" type="revolute">
-    <limit effort="10000" lower="-4.712" upper="4.712" velocity="6.9987"/>
+    <limit effort="10000" lower="-3.14" upper="3.14" velocity="6.9987"/>
        <parent link="RX90_ELBOW" />
        <child link="RX90_FOREARM" />
@@ -196,9 +170,9 @@
        <selfCollide>true</selfCollide>
 	<inertial>
-        <mass value="0.548088"/>
-          <origin xyz="0.000000 -0.000347 0.023671" rpy="0.0 0.0 0.0"/>
-          <inertia ixx="0.000876" ixy="0.000000" ixz="0.000000"
-                                  iyy="0.000889" iyz="0.000005"
-                                                  izz="0.000412"/>
+       <mass value="0.1"/>
+         <origin xyz="0.0 0.00 0.0" rpy="0.0 0.0 0.0"/>
+          <inertia ixx="0.1"  ixy="0.1"  ixz="0.1"
+                   iyx="0.1"  iyy="0.1"  iyz="0.1"
+                   izx="0.1"  izy="0.1"  izz="0.1"/>
     </inertial>
     </link>
@@ -224,10 +198,10 @@
        <selfCollide>true</selfCollide>
 	<inertial>
-        <origin xyz="0 0 0" rpy="0 0 0" />
-         <mass value="0.038484"/>
-          <origin xyz="-0.000245 0.000000 -0.007626" rpy="0.0 0.0 0.0"/>
-          <inertia ixx="0.000011" ixy="0.000000" ixz="0.000000"
-                                  iyy="0.000011" iyz="0.000000"
-                                                  izz="0.000021"/>
+         <origin xyz="0 0 0" rpy="0 0 0" />
+         <mass value="0.1"/>
+        <origin xyz="0.0 0.00 0.0" rpy="0.0 0.0 0.0"/>
+          <inertia ixx="0.1"  ixy="0.1"  ixz="0.1"
+                   iyx="0.1"  iyy="0.1"  iyz="0.1"
+                   izx="0.1"  izy="0.1"  izz="0.1"/>
     </inertial>
     </link>
@@ -253,13 +227,13 @@
        <selfCollide>true</selfCollide>
 	<inertial>
-        <origin xyz="0 0 0" rpy="0 0 0" />
-         <mass value="0.018484"/>
-          <inertia ixx="0.000011" ixy="0.000000" ixz="0.000000"
-                                  iyy="0.000011" iyz="0.000000"
-                                                  izz="0.000021"/>
+        <mass value="0.1" />
+  <origin xyz="0.0 0.00 0.0" rpy="0.0 0.0 0.0"/>
+          <inertia ixx="0.1"  ixy="0.1"  ixz="0.1"
+                   iyx="0.1"  iyy="0.1"  iyz="0.1"
+                   izx="0.1"  izy="0.1"  izz="0.1"/>
     </inertial>
     </link>
     <joint name="RX90_LGRIPPER_JOINT" type="prismatic">
-    <limit effort="1000.0" lower="0" upper="0.1" velocity="0.5"/>
+    <limit effort="100000.0" lower="-0.01" upper="0.08" velocity="20"/>
        <parent link="RX90_FLANGE" />
        <child link="RX90_LGRIPPER" />
@@ -281,13 +255,13 @@
        <selfCollide>true</selfCollide>
 	<inertial>
-        <origin xyz="0 0 0" rpy="0 0 0" />
-         <mass value="0.018484"/>
-          <inertia ixx="0.000011" ixy="0.000000" ixz="0.000000"
-                                  iyy="0.000011" iyz="0.000000"
-                                                  izz="0.000021"/>
+       <origin xyz="0 0 0" rpy="0 0 0" />
+        <mass value="0.1" />
+          <inertia ixx="0.1"  ixy="0.1"  ixz="0.1"
+                   iyx="0.1"  iyy="0.1"  iyz="0.1"
+                   izx="0.1"  izy="0.1"  izz="0.1"/>
     </inertial>
     </link>
     <joint name="RX90_RGRIPPER_JOINT" type="prismatic">
-    <limit effort="1000.0" lower="-0.1" upper="0" velocity="0.5"/>
+    <limit effort="100000.0" lower="-0.08" upper="0.01" velocity="20"/>
        <parent link="RX90_FLANGE" />
        <child link="RX90_RGRIPPER" />
@@ -309,13 +283,13 @@
        <selfCollide>true</selfCollide>
 	<inertial>
-        <origin xyz="0 0 0" rpy="0 0 0" />
-         <mass value="0.018484"/>
-          <inertia ixx="0.000011" ixy="0.000000" ixz="0.000000"
-                                  iyy="0.000011" iyz="0.000000"
-                                                  izz="0.000021"/>
+       <origin xyz="0 0 0" rpy="0 0 0" />
+        <mass value="0.1" />
+          <inertia ixx="0.1"  ixy="0.1"  ixz="0.1"
+                   iyx="0.1"  iyy="0.1"  iyz="0.1"
+                   izx="0.1"  izy="0.1"  izz="0.1"/>
     </inertial>
     </link>
     <joint name="RX90_MGRIPPER_JOINT" type="prismatic">
-    <limit effort="1000.0" lower="-0.05" upper="0" velocity="0.5"/>
+    <limit effort="100000.0" lower="-0.08" upper="0.01" velocity="20"/>
        <parent link="RX90_FLANGE" />
        <child link="RX90_MGRIPPER" />

Commit message: gripper_plugin v3

File: rx90_description/urdf/rx90_floor_baselink.xacro (robot description, xacro)
@@ -235,5 +235,5 @@
     </link>
     <joint name="RX90_LGRIPPER_JOINT" type="prismatic">
-    <limit effort="100000.0" lower="-0.01" upper="0.08" velocity="20"/>
+    <limit effort="100000.0" lower="-0.01" upper="0.018" velocity="20"/>
        <parent link="RX90_FLANGE" />
        <child link="RX90_LGRIPPER" />
@@ -263,5 +263,5 @@
     </link>
     <joint name="RX90_RGRIPPER_JOINT" type="prismatic">
-    <limit effort="100000.0" lower="-0.08" upper="0.01" velocity="20"/>
+    <limit effort="100000.0" lower="-0.02" upper="0.01" velocity="20"/>
        <parent link="RX90_FLANGE" />
        <child link="RX90_RGRIPPER" />
@@ -291,5 +291,5 @@
     </link>
     <joint name="RX90_MGRIPPER_JOINT" type="prismatic">
-    <limit effort="100000.0" lower="-0.08" upper="0.01" velocity="20"/>
+    <limit effort="100000.0" lower="-0.03" upper="0.01" velocity="20"/>
        <parent link="RX90_FLANGE" />
        <child link="RX90_MGRIPPER" />

File: rx90_description/urdf/rx90_floor_noinertia.xacro (robot description, xacro)
@@ -235,5 +235,5 @@
     </link>
     <joint name="RX90_LGRIPPER_JOINT" type="prismatic">
-    <limit effort="100000.0" lower="-0.01" upper="0.08" velocity="20"/>
+    <limit effort="100000.0" lower="-0.01" upper="0.018" velocity="20"/>
        <parent link="RX90_FLANGE" />
        <child link="RX90_LGRIPPER" />
@@ -263,5 +263,5 @@
     </link>
     <joint name="RX90_RGRIPPER_JOINT" type="prismatic">
-    <limit effort="100000.0" lower="-0.08" upper="0.01" velocity="20"/>
+    <limit effort="100000.0" lower="-0.02" upper="0.01" velocity="20"/>
        <parent link="RX90_FLANGE" />
        <child link="RX90_RGRIPPER" />
@@ -291,5 +291,5 @@
     </link>
     <joint name="RX90_MGRIPPER_JOINT" type="prismatic">
-    <limit effort="100000.0" lower="-0.08" upper="0.01" velocity="20"/>
+    <limit effort="100000.0" lower="-0.03" upper="0.01" velocity="20"/>
        <parent link="RX90_FLANGE" />
        <child link="RX90_MGRIPPER" />

Commit message: gripper works

File: rx90_description/urdf/rx90_floor_baselink.xacro (robot description, xacro)
@@ -235,5 +235,5 @@
     </link>
     <joint name="RX90_LGRIPPER_JOINT" type="prismatic">
-    <limit effort="100000.0" lower="-0.01" upper="0.018" velocity="20"/>
+    <limit effort="100000.0" lower="-0.02" upper="0.0" velocity="20"/>
        <parent link="RX90_FLANGE" />
        <child link="RX90_LGRIPPER" />
@@ -263,5 +263,5 @@
     </link>
     <joint name="RX90_RGRIPPER_JOINT" type="prismatic">
-    <limit effort="100000.0" lower="-0.02" upper="0.01" velocity="20"/>
+    <limit effort="100000.0" lower="-0.01" upper="0.02" velocity="20"/>
        <parent link="RX90_FLANGE" />
        <child link="RX90_RGRIPPER" />
@@ -291,5 +291,5 @@
     </link>
     <joint name="RX90_MGRIPPER_JOINT" type="prismatic">
-    <limit effort="100000.0" lower="-0.03" upper="0.01" velocity="20"/>
+    <limit effort="100000.0" lower="-0.01" upper="0.02" velocity="20"/>
        <parent link="RX90_FLANGE" />
        <child link="RX90_MGRIPPER" />

File: rx90_description/urdf/rx90_floor_noinertia.xacro (robot description, xacro)
@@ -235,5 +235,5 @@
     </link>
     <joint name="RX90_LGRIPPER_JOINT" type="prismatic">
-    <limit effort="100000.0" lower="-0.01" upper="0.018" velocity="20"/>
+    <limit effort="100000.0" lower="-0.02" upper="0.0" velocity="20"/>
        <parent link="RX90_FLANGE" />
        <child link="RX90_LGRIPPER" />
@@ -263,5 +263,5 @@
     </link>
     <joint name="RX90_RGRIPPER_JOINT" type="prismatic">
-    <limit effort="100000.0" lower="-0.02" upper="0.01" velocity="20"/>
+    <limit effort="100000.0" lower="-0.01" upper="0.02" velocity="20"/>
        <parent link="RX90_FLANGE" />
        <child link="RX90_RGRIPPER" />
@@ -291,8 +291,36 @@
     </link>
     <joint name="RX90_MGRIPPER_JOINT" type="prismatic">
-    <limit effort="100000.0" lower="-0.03" upper="0.01" velocity="20"/>
+    <limit effort="100000.0" lower="-0.01" upper="0.02" velocity="20"/>
        <parent link="RX90_FLANGE" />
        <child link="RX90_MGRIPPER" />
        <origin rpy="0 ${pi/2} ${-pi/2}" xyz="0.025 0 -0.035" />
+    </joint>
+      <link name="RX90_END">
+       <visual>
+	<origin rpy="0 0 0" xyz="0 0 0" />
+          <geometry>
+            <box size="0.0005 0.0005 0.0005"/>
+          </geometry>
+       </visual>
+	<!--collision>
+        <origin rpy="0 0 0" xyz="0 0 0" />
+            <geometry>
+              <box size="0.0000000000000000000000000000005 0.00000000000000000000005 0.0000000000000000000000000000005"/>
+            </geometry>
+       </collision>
+       <selfCollide>1</selfCollide-->
+	<inertial>
+       <origin xyz="0 0 0" rpy="0 0 0" />
+        <mass value="0.1" />
+          <inertia ixx="0.1"  ixy="0.1"  ixz="0.1"
+                   iyx="0.1"  iyy="0.1"  iyz="0.1"
+                   izx="0.1"  izy="0.1"  izz="0.1"/>
+    </inertial>
+    </link>
+    <joint name="RX90_END_JOINT" type="prismatic">
+    <limit effort="100000.0" lower="-0.03" upper="0.01" velocity="20"/>
+       <parent link="RX90_FLANGE" />
+       <child link="RX90_END" />
+       <origin rpy="0 ${pi/2} ${-pi/2}" xyz="0.025 0.01 0.002" />
     </joint>
 <!--BRAZOOOOOOOOOOOOOOOOOOOOooooooooooooooooooooooooooooooooooooooo-->
@@ -389,3 +417,13 @@
     </actuator>
   </transmission>
+      <transmission name="tran_RX90_END_JOINT">
+    <type>transmission_interface/SimpleTransmission</type>
+    <joint name="RX90_END_JOINT">
+      <hardwareInterface>hardware_interface/EffortJointInterface</hardwareInterface>
+    </joint>
+    <actuator name="motor_RX90_END_JOINT">
+      <hardwareInterface>hardware_interface/EffortJointInterface</hardwareInterface>
+      <mechanicalReduction>1</mechanicalReduction>
+    </actuator>
+  </transmission>
 </robot>
